Commit message: reoriented ird435 pcl

File: husky_ws/src/ur5/ur5_description/urdf/ur5_d435.urdf.xacro (robot description, xacro)
@@ -43,6 +43,7 @@
     <child link="d435_link"/>
   </joint>
-  <xacro:sensor_d435 parent="d435_link" name="intel_cam_" >
+  <xacro:sensor_d435 parent="d435_link" name="intel_cam" >
     <origin xyz="-0.05 -0.01 0.01" rpy="1.57 0 3.14"/>
+     <!-- <origin xyz="0.20 0 0" rpy="0 0 0"/> -->
   </xacro:sensor_d435>
   <!-- Equivalent to the OpenRAVE manipulator denso_robotiq_85_gripper -->
@@ -82,3 +83,44 @@
     </gripper>
   </gazebo>
+  <gazebo reference="intel_cam_link">
+  <sensor name="d435_link_camera" type="depth">
+    <update_rate>20</update_rate>
+    <camera>
+      <horizontal_fov>1.047198</horizontal_fov>
+      <image>
+        <width>640</width>
+        <height>480</height>
+        <format>R8G8B8</format>
+      </image>
+      <clip>
+        <near>0.05</near>
+        <far>3</far>
+      </clip>
+    </camera>
+    <plugin name="d435_link_controller" filename="libgazebo_ros_openni_kinect.so">
+      <baseline>0.2</baseline>
+      <alwaysOn>true</alwaysOn>
+      <updateRate>1.0</updateRate>
+      <cameraName>intel_cam_ir</cameraName>
+      <imageTopicName>/intel_cam/color/image_raw</imageTopicName>
+      <cameraInfoTopicName>/intel_cam/color/camera_info</cameraInfoTopicName>
+      <depthImageTopicName>/intel_cam/depth/image_raw</depthImageTopicName>
+      <depthImageInfoTopicName>/intel_cam/depth/camera_info</depthImageInfoTopicName>
+      <pointCloudTopicName>/intel_cam/depth/points</pointCloudTopicName>
+      <frameName>intel_cam_depth_optical_frame</frameName>
+      <pointCloudCutoff>0.5</pointCloudCutoff>
+      <pointCloudCutoffMax>3.0</pointCloudCutoffMax>
+      <distortionK1>0.00000001</distortionK1>
+      <distortionK2>0.00000001</distortionK2>
+      <distortionK3>0.00000001</distortionK3>
+      <distortionT1>0.00000001</distortionT1>
+      <distortionT2>0.00000001</distortionT2>
+      <CxPrime>0</CxPrime>
+      <Cx>0</Cx>
+      <Cy>0</Cy>
+      <focalLength>0</focalLength>
+      <hackBaseline>0</hackBaseline>
+    </plugin>
+  </sensor>
+</gazebo>
 </robot>

Commit message: pcl works and planner has no collision between camera and wrist

File: husky_ws/src/ur5/ur5_description/urdf/ur5_d435.urdf.xacro (robot description, xacro)
@@ -44,5 +44,5 @@
   </joint>
   <xacro:sensor_d435 parent="d435_link" name="intel_cam" >
-    <origin xyz="-0.05 -0.01 0.01" rpy="1.57 0 3.14"/>
+    <origin xyz="-0.10 -0.01 0.01" rpy="1.57 0 3.14"/>
      <!-- <origin xyz="0.20 0 0" rpy="0 0 0"/> -->
   </xacro:sensor_d435>
