Commit message: added namespaces in octomap

File: husky_ws/src/ur5/ur5_description/urdf/ur5_d435_with_prints.urdf.xacro (robot description, xacro)
@@ -88,5 +88,5 @@
   </joint>
   <xacro:sensor_d435 parent="d435_link" name="intel_cam" >
-    <origin xyz="-0.08 -0.01 0.01" rpy="1.57 0 3.14"/>
+    <origin xyz="-0.06 -0.01 -0.01" rpy="1.57 0 3.14"/>
      <!-- <origin xyz="0.20 0 0" rpy="0 0 0"/> -->
   </xacro:sensor_d435>
