Commit message: added velodyne lidar

File: husky_ws/src/husky/husky_description/urdf/husky.urdf.xacro (robot description, xacro)
@@ -42,4 +42,5 @@
   <xacro:include filename="$(find husky_description)/urdf/accessories/sensor_arch.urdf.xacro"/>
   <xacro:include filename="$(find ur5_description)/urdf/ur5_robotiq85_gripper.urdf.xacro" />
+  <xacro:include filename="$(find velodyne_description)/urdf/VLP-16.urdf.xacro" />
   <!--<xacro:include filename="$(find robotiq_2f_85_gripper_visualization)/urdf/robotiq_arg2f_85_model_macro.xacro" />-->
   <!--<xacro:include filename="$(find ur_description)/urdf/ur5_joint_limited_robot.urdf.xacro" />-->
@@ -122,4 +123,10 @@
   </xacro:husky_wheel>
   <xacro:husky_decorate />
+  <xacro:arg name="gpu" default="false"/>
+  <xacro:property name="gpu" value="$(arg gpu)" />
+  <xacro:include filename="$(find velodyne_description)/urdf/VLP-16.urdf.xacro"/>
+  <VLP-16 parent="top_plate_link" name="velodyne" topic="/velodyne_points" hz="10" samples="440" gpu="${gpu}">
+    <origin xyz="0.30 0 0.0" rpy="0 0 0" />
+  </VLP-16>
   <xacro:if value="$(arg laser_enabled)">
     <sick_lms1xx_mount prefix="base"/>
@@ -142,5 +149,5 @@
     <xacro:property name="reflect" value="-1" />
     <joint name="ur5_arm_base" type="fixed">
-      <origin xyz="0.3058 0 0.0065" rpy="0.0 0.0 -1.57" />
+      <origin xyz="-0.05 0 0.0065" rpy="0.0 0.0 -1.57" />
       <parent link="top_plate_link" />
       <child link="ur5_arm_base_link"/>

Commit message: bf cleanup

File: husky_ws/src/husky/husky_description/urdf/husky.urdf.xacro (robot description, xacro)
@@ -140,5 +140,5 @@
   <xacro:if value="$(arg kinect_enabled)">
     <joint name="kinect_frame_joint" type="fixed">
-      <origin xyz="0.4 0.0 -0.10" rpy="0.0 0.0 0.0" />
+      <origin xyz="0.35 0.0 -0.20" rpy="0.0 0.0 0.0" />
       <parent link="top_plate_link" />
       <child link="camera_link"/>
@@ -149,5 +149,5 @@
     <xacro:property name="reflect" value="-1" />
     <joint name="ur5_arm_base" type="fixed">
-      <origin xyz="-0.05 0 0.0065" rpy="0.0 0.0 -1.57" />
+      <origin xyz="-0.30 0 0.0065" rpy="0.0 0.0 1.57" />
       <parent link="top_plate_link" />
       <child link="ur5_arm_base_link"/>

Commit message: no stl for now, but ird435 in reasonable distance

File: husky_ws/src/husky/husky_description/urdf/husky.urdf.xacro (robot description, xacro)
@@ -42,5 +42,5 @@
   <xacro:include filename="$(find husky_description)/urdf/accessories/sensor_arch.urdf.xacro"/>
   <!--<xacro:include filename="$(find ur5_description)/urdf/ur5_robotiq85_gripper.urdf.xacro" />-->
-  <xacro:include filename="$(find ur5_description)/urdf/ur5_d435.urdf.xacro" />
+  <xacro:include filename="$(find ur5_description)/urdf/ur5_d435_with_prints.urdf.xacro" />
   <xacro:include filename="$(find velodyne_description)/urdf/VLP-16.urdf.xacro" />
   <!--<xacro:include filename="$(find robotiq_2f_85_gripper_visualization)/urdf/robotiq_arg2f_85_model_macro.xacro" />-->
@@ -141,5 +141,5 @@
   <xacro:if value="$(arg kinect_enabled)">
     <joint name="kinect_frame_joint" type="fixed">
-      <origin xyz="0.35 0.0 -0.20" rpy="0.0 0.0 0.0" />
+      <origin xyz="0.3 0.0 -0.07" rpy="0.0 0.40 0.0" />
       <parent link="top_plate_link" />
       <child link="camera_link"/>
